Commit message: fixed location of origin

File: hector_quadrotor_sim/hector_quadrotor/hector_quadrotor_description/urdf/quadrotor_base.urdf.xacro (robot description, xacro)
@@ -13,4 +13,5 @@
       <visual>
         <origin xyz="0 0 0" rpy="0 0 0" />
+        <!-- <origin xyz="28.204388 7.095104 -9.95" rpy="0 0 0" /> -->
         <geometry>
           <mesh filename="package://hector_quadrotor_description/meshes/quadrotor/quadrotor_base.dae"/>

Commit message: changed scale of appearance for quadrotor model by 3x. spawn position for quadrotor is now on top of helipad.

File: hector_quadrotor_sim/hector_quadrotor/hector_quadrotor_description/urdf/quadrotor_base.urdf.xacro (robot description, xacro)
@@ -15,5 +15,5 @@
         <!-- <origin xyz="28.204388 7.095104 -9.95" rpy="0 0 0" /> -->
         <geometry>
-          <mesh filename="package://hector_quadrotor_description/meshes/quadrotor/quadrotor_base.dae"/>
+          <mesh filename="package://hector_quadrotor_description/meshes/quadrotor/quadrotor_base.dae" scale = "3 3 3"/>
         </geometry>
       </visual>
@@ -21,5 +21,5 @@
         <origin xyz="0 0 0" rpy="0 0 0" />
         <geometry>
-          <mesh filename="package://hector_quadrotor_description/meshes/quadrotor/quadrotor_base.stl"/>
+          <mesh filename="package://hector_quadrotor_description/meshes/quadrotor/quadrotor_base.stl" scale = "3 3 3"/>
         </geometry>
       </collision>

Commit message: started trying to upscale model mass and propulsion output by 4 so they will be balanced. not working currently.

File: hector_quadrotor_sim/hector_quadrotor/hector_quadrotor_description/urdf/quadrotor_base.urdf.xacro (robot description, xacro)
@@ -4,5 +4,6 @@
   <xacro:property name="pi" value="3.1415926535897931" />
   <!-- Main quadrotor link -->
-  <xacro:macro name="quadrotor_base_macro">
+  <!-- Old Values pre-upscaling -->
+  <!-- <xacro:macro name="quadrotor_base_macro">
     <link name="base_link">
       <inertial>
@@ -10,4 +11,11 @@
         <origin xyz="0 0 0" />
         <inertia ixx="0.01152" ixy="0.0" ixz="0.0" iyy="0.01152" iyz="0.0" izz="0.0218" />
+      </inertial> -->
+  <xacro:macro name="quadrotor_base_macro">
+    <link name="base_link">
+      <inertial>
+        <mass value="5.908" />
+        <origin xyz="0 0 0" />
+        <inertia ixx="0.04608" ixy="0.0" ixz="0.0" iyy="0.04608" iyz="0.0" izz="0.0872" />
       </inertial>
       <visual>
@@ -15,5 +23,5 @@
         <!-- <origin xyz="28.204388 7.095104 -9.95" rpy="0 0 0" /> -->
         <geometry>
-          <mesh filename="package://hector_quadrotor_description/meshes/quadrotor/quadrotor_base.dae" scale = "3 3 3"/>
+          <mesh filename="package://hector_quadrotor_description/meshes/quadrotor/quadrotor_base.dae" scale = "4 4 4"/>
         </geometry>
       </visual>
@@ -21,5 +29,5 @@
         <origin xyz="0 0 0" rpy="0 0 0" />
         <geometry>
-          <mesh filename="package://hector_quadrotor_description/meshes/quadrotor/quadrotor_base.stl" scale = "3 3 3"/>
+          <mesh filename="package://hector_quadrotor_description/meshes/quadrotor/quadrotor_base.stl" scale = "4 4 4"/>
         </geometry>
       </collision>

Commit message: james upscaling first attempt  - in quadrotor urdf file: mass from 1.477 to 5.0  - scaled inertia and controller.yaml force limits by same factor  - changed navigation file to citynavigation in launch  - changed force amplitude to 0 to test without forces

File: hector_quadrotor_sim/hector_quadrotor/hector_quadrotor_description/urdf/quadrotor_base.urdf.xacro (robot description, xacro)
@@ -7,7 +7,10 @@
     <link name="base_link">
       <inertial>
-        <mass value="1.477" />
+        <!-- commented lines are previous values-->
+        <!-- <mass value="1.477" /> -->
+        <mass value="5.0" />
         <origin xyz="0 0 0" />
-        <inertia ixx="0.01152" ixy="0.0" ixz="0.0" iyy="0.01152" iyz="0.0" izz="0.0218" />
+        <!-- <inertia ixx="0.01152" ixy="0.0" ixz="0.0" iyy="0.01152" iyz="0.0" izz="0.0218" /> -->
+        <inertia ixx="0.03905" ixy="0.0" ixz="0.0" iyy="0.03905" iyz="0.0" izz="0.0739" />
       </inertial>
       <visual>

Commit message: Changed quadrotor weight to 6500kg and scaled inertia and controller limits along with it. drone can almost handle 608N of torque now but still needs some CS tuning

File: hector_quadrotor_sim/hector_quadrotor/hector_quadrotor_description/urdf/quadrotor_base.urdf.xacro (robot description, xacro)
@@ -9,8 +9,8 @@
         <!-- commented lines are previous values-->
         <!-- <mass value="1.477" /> -->
-        <mass value="5.0" />
+        <mass value="6500.0" />
         <origin xyz="0 0 0" />
         <!-- <inertia ixx="0.01152" ixy="0.0" ixz="0.0" iyy="0.01152" iyz="0.0" izz="0.0218" /> -->
-        <inertia ixx="0.03905" ixy="0.0" ixz="0.0" iyy="0.03905" iyz="0.0" izz="0.0739" />
+        <inertia ixx="50.69735952" ixy="0.0" ixz="0.0" iyy="50.69735952" iyz="0.0" izz="95.93771158" />
       </inertial>
       <visual>
@@ -18,5 +18,5 @@
         <!-- <origin xyz="28.204388 7.095104 -9.95" rpy="0 0 0" /> -->
         <geometry>
-          <mesh filename="package://hector_quadrotor_description/meshes/quadrotor/quadrotor_base.dae" scale = "3 3 3"/>
+          <mesh filename="package://hector_quadrotor_description/meshes/quadrotor/quadrotor_base.dae" scale = "4 4 4"/>
         </geometry>
       </visual>
@@ -24,5 +24,5 @@
         <origin xyz="0 0 0" rpy="0 0 0" />
         <geometry>
-          <mesh filename="package://hector_quadrotor_description/meshes/quadrotor/quadrotor_base.stl" scale = "3 3 3"/>
+          <mesh filename="package://hector_quadrotor_description/meshes/quadrotor/quadrotor_base.stl" scale = "4 4 4"/>
         </geometry>
       </collision>
